Commit message: delete unnecessary scenes

File: urdf/scene_D.xacro (robot description, xacro)
@@ -64,5 +64,5 @@
       </visual>
       <collision>
-        <origin xyz="0.004 0.029 0" rpy="1.5708 0 0"/>
+        <origin xyz="0 0 0" rpy="-1.5708 0 0"/>
         <geometry>
           <mesh filename="package://suction-gripper/meshes/collision/Gripper_Suction_collision.STL" scale="0.001 0.001 0.001"/>

File: urdf/ur5e_sgripper.urdf.xacro (robot description, xacro)
@@ -7,5 +7,5 @@
     <xacro:include filename="$(find ur_description)/urdf/ur5e.xacro" />
     <!--  Tables and Walls -->
-    <xacro:include filename="$(find apple_proxy)/urdf/scene_D.xacro" />
+    <xacro:include filename="$(find suction-gripper)/urdf/scene_D.xacro" />
     <xacro:tables />
     <!-- STEP 2: DEFINE THE INTERFACES AMONG ALL THE LINKS FROM -->
@@ -17,6 +17,5 @@
     <parent link="tool0" />
     <child link="suction_gripper" />
-    <origin xyz="-0.026 -0.039 0.175" rpy="-1.5708 0 0" />
-        <!-- Note: x and y offset is because the cframe of the 3d model is not located in the center -->
+    <origin xyz="0 0 0.15" rpy="1.5708 0 0" />
     </joint>
     <!-- Describe the interface between the world and the tables -->

Commit message: config

File: urdf/scene_D.xacro (robot description, xacro)
@@ -19,5 +19,22 @@
       </collision>
     </link>
-    <link name="joes_ur5_table" >
+    <link name="small_table" >
+      <visual>
+        <origin xyz="0 0 0" rpy="0 0 0"/>
+        <geometry>
+          <mesh filename="package://apple_proxy/meshes/furniture/collision/UR5_small_table.STL" scale="0.001 0.001 0.001"/>
+        </geometry>
+        <material name="Grey">
+          <color rgba="0.5 0.5 0.5 1.0"/>
+        </material>
+      </visual>
+      <collision>
+        <origin xyz="0 0 0" rpy="0 0 0"/>
+        <geometry>
+          <mesh filename="package://apple_proxy/meshes/furniture/collision/UR5_small_table.STL" scale="0.001 0.001 0.001"/>
+        </geometry>
+      </collision>
+    </link>
+    <!-- <link name="joes_ur5_table" >
       <visual>
         <origin xyz="0 0 0" rpy="0 0 0"/>
@@ -35,5 +52,5 @@
         </geometry>
       </collision>
-    </link>
+    </link>     -->
     <!-- <link name="test_rig" >
       <visual>
@@ -70,4 +87,21 @@
       </collision>
     </link>
+    <link name="apple_proxy">
+      <visual>
+        <origin xyz="-0.11498 0.7701 0" rpy="0 0 -1.5708"/>
+        <geometry>
+          <mesh filename="package://apple_proxy/meshes/apple_proxy/visual/apple_proxy_visual.STL" scale="0.001 0.001 0.001"/>
+        </geometry>
+        <material name="Green">
+          <color rgba="0 1 0 0.7"/>
+        </material>
+      </visual>
+      <collision>
+        <origin xyz="0 0 0" rpy="0 0 0"/>
+        <geometry>
+          <mesh filename="package://apple_proxy/meshes/apple_proxy/collision/apple_proxy_collision.STL" scale="0.001 0.001 0.001"/>
+        </geometry>
+      </collision>
+    </link>
   </xacro:macro>
 </robot>

File: urdf/ur5e_sgripper.urdf.xacro (robot description, xacro)
@@ -17,5 +17,5 @@
     <parent link="tool0" />
     <child link="suction_gripper" />
-    <origin xyz="0 0 0.15" rpy="1.5708 0 0" />
+    <origin xyz="0 0 0.162" rpy="1.5708 0 0" />
     </joint>
     <!-- Describe the interface between the world and the tables -->
@@ -27,12 +27,18 @@
     <joint name="world_small_table" type="fixed">
     <parent link="world" />
-    <child link="joes_ur5_table" />
-    <origin xyz="0.915 0.097 0.7660" rpy="-3.1416 0 3.1416" />
+    <child link="small_table" />
+    <origin xyz="-0.29 -1.57 0" rpy="0 0 1.5708" />
+    </joint>
+    <!-- Describe the interface between the world and the Apple Proxy -->
+    <joint name = "bigTable_simpleProxy" type="fixed">
+    <parent link = "big_table" />
+    <child link = "apple_proxy" />
+    <origin xyz = "0.4572 0.91 0.895" rpy="1.5708 0 -1.5708" />
     </joint>
     <!-- Describe the interface between the world and the robot" -->
     <joint name="world_joint" type="fixed">
-    <parent link="joes_ur5_table" />
+    <parent link="small_table" />
     <child link = "base_link" />
-    <origin xyz="0.71 0.25 0" rpy="3.1416 0.0 -0.7854" />
+    <origin xyz="0.358 0.357 0.858" rpy="0.0 0.0 3.1416" />
     </joint>
     <!-- Describe the location of the tip of the suction gripper -->
