Commit message: urdf

File: urdf/ur5e_sgripper.urdf.xacro (robot description, xacro)
@@ -7,14 +7,14 @@
     <xacro:include filename="$(find ur_description)/urdf/ur5e.xacro" />
     <!--  Tables and Walls -->
-    <xacro:include filename="$(find apple_proxy)/urdf/scene_C.xacro" />
+    <xacro:include filename="$(find apple_proxy)/urdf/scene_D.xacro" />
     <xacro:tables />
     <!-- STEP 2: DEFINE THE INTERFACES AMONG ALL THE LINKS FROM -->
     <!-- Here is where you define the scene and how the cframes are related -->
-    <link name="world" />
-    <link name="suction_cup" />
+    <link name="world"  />
+    <link name="eef" doc="point at ___cm from the palm"    />
     <!-- Describe the interface between the robot and the gripper -->
     <joint name="robotiq_coupler_joint" type="fixed">
     <parent link="tool0" />
-    <child link="test_rig" />
+    <child link="suction_gripper" />
     <origin xyz="-0.026 -0.039 0.175" rpy="-1.5708 0 0" />
         <!-- Note: x and y offset is because the cframe of the 3d model is not located in the center -->
@@ -31,10 +31,4 @@
     <origin xyz="0.915 0.097 0.7660" rpy="-3.1416 0 3.1416" />
     </joint>
-    <!-- Describe the interface between the world and the Semi sphere -->
-    <joint name = "bigTable_simpleProxy" type="fixed"> -->
-    <parent link = "big_table" /> -->
-    <child link = "sphere" /> -->
-    <origin xyz = "0.115 0 1.0325" rpy="0 3.1416 0" />
-    </joint>
     <!-- Describe the interface between the world and the robot" -->
     <joint name="world_joint" type="fixed">
@@ -44,14 +38,8 @@
     </joint>
     <!-- Describe the location of the tip of the suction cup -->
-    <joint name="suction_cup" type="fixed">
-    <parent link="tool0" />
-    <child link="suction_cup" />
+    <joint name="ideal_eef" type="fixed">
+    <parent link="suction_gripper" />
+    <child link="eef" />
     <origin xyz="0 0 0.203" rpy="0 0 0" />
     </joint>
-    <!-- Describe the location of the tip of the suction cup -->
-    <joint name="suction_cup_model" type="fixed">
-    <parent link="tool0" />
-    <child link="suction_cup_model" />
-    <origin xyz="-0.0165 0.0165 0.203" rpy="3.1416 0 0" />
-    </joint>
 </robot>

Commit message: config

File: urdf/ur5e_sgripper.urdf.xacro (robot description, xacro)
@@ -36,9 +36,9 @@
     <origin xyz="0.71 0.25 0" rpy="3.1416 0.0 -0.7854" />
     </joint>
-    <!-- Describe the location of the tip of the suction cup -->
+    <!-- Describe the location of the tip of the suction gripper -->
     <joint name="ideal_eef" type="fixed">
     <parent link="suction_gripper" />
     <child link="eef" />
-    <origin xyz="0 0 0.203" rpy="0 0 0" />
+    <origin xyz="0 0.02 0" rpy="-1.5708 0 0" />
     </joint>
 </robot>

Commit message: arduino libraries upgrade

File: urdf/ur5e_sgripper.urdf.xacro (robot description, xacro)
@@ -28,5 +28,5 @@
     <parent link="world" />
     <child link="small_table" />
-    <origin xyz="-0.29 -1.57 0" rpy="0 0 1.5708" />
+    <origin xyz="-0.29 -1.30 0" rpy="0 0 1.5708" />
     </joint>
     <!-- Describe the interface between the world and the Apple Proxy -->

Commit message: Apple pose calibration for demos!

File: urdf/ur5e_sgripper.urdf.xacro (robot description, xacro)
@@ -28,5 +28,5 @@
     <parent link="world" />
     <child link="small_table" />
-    <origin xyz="-0.29 -1.30 0" rpy="0 0 1.5708" />
+    <origin xyz="-0.155 -1.65 0" rpy="0 0 1.5708" />
     </joint>
     <!-- Describe the interface between the world and the Apple Proxy -->

Commit message: added script to sample points in a 2d

File: urdf/ur5e_sgripper.urdf.xacro (robot description, xacro)
@@ -28,5 +28,7 @@
     <parent link="world" />
     <child link="small_table" />
-    <origin xyz="-0.155 -1.65 0" rpy="0 0 1.5708" />
+    <origin xyz="-0.155 -1.45 0" rpy="0 0 1.5708" />
+    <!-- <origin xyz="-0.155 -1.50 0" rpy="0 0 1.5708" /> -->
+    <!-- <origin xyz="-0.155 -1.65 0" rpy="0 0 1.5708" />    -->
     </joint>
     <!-- Describe the interface between the world and the Apple Proxy -->

Commit message: Fixed location of robot w.r.t small table

File: urdf/ur5e_sgripper.urdf.xacro (robot description, xacro)
@@ -42,5 +42,5 @@
     <parent link="small_table" />
     <child link = "base_link" />
-    <origin xyz="0.358 0.357 0.858" rpy="0.0 0.0 3.1416" />
+    <origin xyz="0.255 0.357 0.858" rpy="0.0 0.0 3.1416" />
     </joint>
     <!-- Describe the location of the tip of the suction gripper -->

Commit message: Fixed location of robot w.r.t small table

File: urdf/ur5e_sgripper.urdf.xacro (robot description, xacro)
@@ -28,5 +28,5 @@
     <parent link="world" />
     <child link="small_table" />
-    <origin xyz="-0.155 -1.45 0" rpy="0 0 1.5708" />
+    <origin xyz="-0.155 -1.35 0" rpy="0 0 1.5708" />
     <!-- <origin xyz="-0.155 -1.50 0" rpy="0 0 1.5708" /> -->
     <!-- <origin xyz="-0.155 -1.65 0" rpy="0 0 1.5708" />    -->

Commit message: apple z depending on the type of stem, because it varies a bit

File: urdf/ur5e_sgripper.urdf.xacro (robot description, xacro)
@@ -17,5 +17,5 @@
     <parent link="tool0" />
     <child link="suction_gripper" />
-    <origin xyz="0 0 0.162" rpy="1.5708 0 0" />
+    <origin xyz="0 0 0.162" rpy="1.5708 0 0.44" />
     </joint>
     <!-- Describe the interface between the world and the tables -->

Commit message: experiments in lab - Feb 8 2024

File: urdf/ur5e_sgripper.urdf.xacro (robot description, xacro)
@@ -42,5 +42,5 @@
     <parent link="small_table" />
     <child link = "base_link" />
-    <origin xyz="0.255 0.357 0.858" rpy="0.0 0.0 3.1416" />
+    <origin xyz="0.35 0.357 0.858" rpy="0.0 0.0 3.1416" />
     </joint>
     <!-- Describe the location of the tip of the suction gripper -->

Commit message: adjustments for the occlusion trials

File: urdf/ur5e_sgripper.urdf.xacro (robot description, xacro)
@@ -28,5 +28,5 @@
     <parent link="world" />
     <child link="small_table" />
-    <origin xyz="-0.155 -1.35 0" rpy="0 0 1.5708" />
+    <origin xyz="0 -1.35 0" rpy="0 0 1.5708" />
     <!-- <origin xyz="-0.155 -1.50 0" rpy="0 0 1.5708" /> -->
     <!-- <origin xyz="-0.155 -1.65 0" rpy="0 0 1.5708" />    -->
@@ -36,5 +36,5 @@
     <parent link = "big_table" />
     <child link = "apple_proxy" />
-    <origin xyz = "0.4572 0.91 0.895" rpy="1.5708 0 -1.5708" />
+    <origin xyz = "0.4572 0.63 0.895" rpy="1.5708 0 -1.5708" />
     </joint>
     <!-- Describe the interface between the world and the robot" -->
@@ -42,5 +42,5 @@
     <parent link="small_table" />
     <child link = "base_link" />
-    <origin xyz="0.35 0.357 0.858" rpy="0.0 0.0 3.1416" />
+    <origin xyz="0.35 0.357 0.858" rpy="0.0 0.0 0.0" />
     </joint>
     <!-- Describe the location of the tip of the suction gripper -->

Commit message: Adjusted the angle of the gripper w.r.t. tool. The correct value is -15deg (-0.261rad) in YAW

File: urdf/ur5e_sgripper.urdf.xacro (robot description, xacro)
@@ -14,8 +14,9 @@
     <link name="eef" doc="point at ___cm from the palm"    />
     <!-- Describe the interface between the robot and the gripper -->
+    <!-- The gripper is rotated -15deg (-0.261rad) w.r.t. tool -->
     <joint name="robotiq_coupler_joint" type="fixed">
     <parent link="tool0" />
     <child link="suction_gripper" />
-    <origin xyz="0 0 0.162" rpy="1.5708 0 0.44" />
+    <origin xyz="0 0 0.162" rpy="1.5708 0 -0.261" />
     </joint>
     <!-- Describe the interface between the world and the tables -->

Commit message: PressureTese file from Olivia

File: urdf/ur5e_sgripper.urdf.xacro (robot description, xacro)
@@ -46,8 +46,9 @@
     </joint>
     <!-- Describe the location of the tip of the suction gripper -->
+    <!-- Offsets: Originally 2cm -->
     <joint name="ideal_eef" type="fixed">
     <parent link="suction_gripper" />
     <child link="eef" />
-    <origin xyz="0 0.02 0" rpy="-1.5708 0 0" />
+    <origin xyz="0 0 0.6" rpy="-1.5708 0 0" />
     </joint>
 </robot>

Commit message: Update for Pressure Tests: * Location of eef cframe w.r.t. suction gripper cframe:   It is located 6cm in the y axis of the suction gripper cfram.

File: urdf/ur5e_sgripper.urdf.xacro (robot description, xacro)
@@ -46,9 +46,9 @@
     </joint>
     <!-- Describe the location of the tip of the suction gripper -->
-    <!-- Offsets: Originally 2cm -->
+    <!-- Offsets: Originally 2cm (Warning!!! w.r.t. y axis) -->
     <joint name="ideal_eef" type="fixed">
     <parent link="suction_gripper" />
     <child link="eef" />
-    <origin xyz="0 0 0.6" rpy="-1.5708 0 0" />
+    <origin xyz="0 0.06 0" rpy="-1.5708 0 0" />
     </joint>
 </robot>

Commit message: Update for Pressure Tests: * Location of eef cframe w.r.t. suction gripper cframe:   It is located 6cm in the y axis of the suction gripper cfram.

File: urdf/ur5e_sgripper.urdf.xacro (robot description, xacro)
@@ -50,5 +50,5 @@
     <parent link="suction_gripper" />
     <child link="eef" />
-    <origin xyz="0 0.06 0" rpy="-1.5708 0 0" />
+    <origin xyz="0 0.04 0" rpy="-1.5708 0 0" />
     </joint>
 </robot>

Commit message: suction cup cframes for pressure servoing

File: urdf/ur5e_sgripper.urdf.xacro (robot description, xacro)
@@ -13,4 +13,7 @@
     <link name="world"  />
     <link name="eef" doc="point at ___cm from the palm"    />
+    <link name="eef_SCA" doc="point at ___cm from the palm"    />
+    <link name="eef_SCB" doc="point at ___cm from the palm"    />
+    <link name="eef_SCC" doc="point at ___cm from the palm"    />
     <!-- Describe the interface between the robot and the gripper -->
     <!-- The gripper is rotated -15deg (-0.261rad) w.r.t. tool -->
@@ -18,5 +21,5 @@
     <parent link="tool0" />
     <child link="suction_gripper" />
-    <origin xyz="0 0 0.162" rpy="1.5708 0 -0.261" />
+    <origin xyz="0 0 0.177" rpy="1.5708 0 -0.261" />
     </joint>
     <!-- Describe the interface between the world and the tables -->
@@ -50,5 +53,26 @@
     <parent link="suction_gripper" />
     <child link="eef" />
-    <origin xyz="0 0.04 0" rpy="-1.5708 0 0" />
+    <origin xyz="0 0.012 0" rpy="-1.5708 0 0" />
+    </joint>
+    <!-- Describe the location of the suction cups -->
+    <!-- Offsets: Originally 2cm (Warning!!! w.r.t. y axis) -->
+    <joint name="ideal_eef_SCA" type="fixed">
+    <parent link="eef" />
+    <child link="eef_SCA" />
+    <origin xyz="+0.016 +0.027128 0" rpy="0 0 0" />
+    </joint>
+    <!-- Describe the location of the suction cups -->
+    <!-- Offsets: Originally 2cm (Warning!!! w.r.t. y axis) -->
+    <joint name="ideal_eef_SCB" type="fixed">
+    <parent link="eef" />
+    <child link="eef_SCB" />
+    <origin xyz="-0.032 0 0" rpy="0 0 0" />
+    </joint>
+    <!-- Describe the location of the suction cups -->
+    <!-- Offsets: Originally 2cm (Warning!!! w.r.t. y axis) -->
+    <joint name="ideal_eef_SCC" type="fixed">
+    <parent link="eef" />
+    <child link="eef_SCC" />
+    <origin xyz="+0.016 -0.027128 0" rpy="0 0 0" />
     </joint>
 </robot>

Commit message: sequences for experiments

File: urdf/ur5e_sgripper.urdf.xacro (robot description, xacro)
@@ -32,5 +32,5 @@
     <parent link="world" />
     <child link="small_table" />
-    <origin xyz="0 -1.35 0" rpy="0 0 1.5708" />
+    <origin xyz="0 -1.44 0" rpy="0 0 1.5708" />
     <!-- <origin xyz="-0.155 -1.50 0" rpy="0 0 1.5708" /> -->
     <!-- <origin xyz="-0.155 -1.65 0" rpy="0 0 1.5708" />    -->
